File: untitled.kicad_sch (KiCad schematic)
At the start: 66 parts, among them J501 Conn_01x01_Female, J502 Screw_Terminal_01x02, J503 Conn_01x01_Female, J504 Conn_01x03_Male, J505 Conn_01x02_Male, J506 Conn_01x02_Male, J507 Conn_01x02_Male, J508 Conn_01x01_Female, J509 Screw_Terminal_01x02, J510 Conn_01x01_Female, U501 Optical_reciver, U502 Optical_reciver, U503 74HC14, U504 LM311, U505 74HC74, U506 74LS00, U507 TLV7031DBV

Commit message: Update
Parts:
- added D509, D510: LED, symbol Device:LED
- added R515, R516: 470, symbol Device:R
- renumbered D509 to D511, J508 to J501, J509 to J502, J510 to J503, J501 to J504, J502 to J505, J503 to J506, J504 to J507, J505 to J508, J506 to J509, J507 to J510, R515 to R517, R516 to R518, R517 to R519
Connections:
- net GND: now also D509.1 (K), D510.1 (K)
- net LED_inteep: now also R515.2
- net LED_overcurrent: now also R516.2
- new net: D509.2 (A), R515.1
- new net: D510.2 (A), R516.1
