File: DRSSTC.kicad_pcb (KiCad board)
At the start: 2 copper layers, 129 parts, among them J201 Screw_Terminal_01x01, J202 Screw_Terminal_01x01, J301 Screw_Terminal_01x02, J401 Conn_01x01_Female, J402 Screw_Terminal_01x02, J403 Conn_01x01_Female, J404 Conn_01x01_Female, J405 Screw_Terminal_01x02, J406 Conn_01x01_Female, J407 Conn_01x01_Female, J408 Screw_Terminal_01x02, J409 Conn_01x01_Female, J410 Conn_01x01_Female, J411 Screw_Terminal_01x02, J412 Conn_01x01_Female, J413 Conn_01x01_Female, J414 Screw_Terminal_01x02, J415 Conn_01x01_Female, J501 Conn_01x01_Female, J502 Screw_Terminal_01x02, J503 Conn_01x01_Female, J504 Conn_01x03_Male, J505 Conn_01x02_Male, J506 Conn_01x02_Male, J507 Conn_01x02_Male, J508 Conn_01x01_Female, J509 Screw_Terminal_01x02, J510 Conn_01x01_Female, Q201 Q_NMOS_GDS, Q202 Q_NMOS_GDS, Q203 Q_NMOS_GDS, Q204 Q_NMOS_GDS, Q401 Q_PMOS_GDS, Q402 Q_NMOS_GDS, Q403 Q_PMOS_GDS, Q404 Q_NMOS_GDS, U401 UCC27524, U501 Optical_reciver, U502 Optical_reciver, U503 74HC14, U504 LM311, U505 74HC74, U506 74LS00, U507 TLV7031DBV

Commit message: 0.1V control-circuit
Next relese:
Mounting holes;
Fan header;
Better layout;
Bigger  capacitors;
Parts:
- removed D201, D202, D211, D212, D509: D, Diode_SMD:D_0805_2012Metric
- removed D203, D204, D205, D206, D207, D208, D209, D210: D_Zener, Diode_SMD:D_0805_2012Metric
- removed J201, J202: Screw_Terminal_01x01, TerminalBlock_MetzConnect:TerminalBlock_MetzConnect_360271_1x01_Horizontal_ScrewM3.0_Boxed
- removed J404, J406, J407, J409, J410, J412, J413, J415: Conn_01x01_Female, Connector_PinHeader_2.54mm:PinHeader_1x01_P2.54mm_Vertical
- removed J405, J408, J411, J414: Screw_Terminal_01x02, TerminalBlock:TerminalBlock_Altech_AK300-2_P5.00mm
- removed Q201, Q202, Q203, Q204: Q_NMOS_GDS, Package_TO_SOT_THT:TO-247-3_Horizontal_TabUp
- removed R201, R202, R203, R204: 5.1, Resistor_SMD:R_1206_3216Metric
- removed R301: 5.1k, Resistor_SMD:R_0805_2012Metric
- removed R515: 470, Resistor_SMD:R_0805_2012Metric
- removed R516: 100k, Resistor_SMD:R_0805_2012Metric
- removed U501, U502: Optical_reciver, OptoDevice:PLT135
- added D1: D, Diode_SMD:D_0805_2012Metric, F.Cu at (214.4, 106.9)
- added D2: D, Diode_SMD:D_0805_2012Metric, F.Cu at (193.9, 124.9)
- added D3: D, Diode_SMD:D_0805_2012Metric, F.Cu at (170.9, 128.2)
- added D4: D, Diode_SMD:D_0805_2012Metric, F.Cu at (219.0, 102.3)
- added D5: D, Diode_SMD:D_0805_2012Metric, F.Cu at (175.3, 128.2)
- added D511: LL4148, Diode_SMD:D_0805_2012Metric, F.Cu at (321.6, 29.5)
- added D6: D, Diode_SMD:D_0805_2012Metric, F.Cu at (200.5, 120.3)
- added D7: D, Diode_SMD:D_0805_2012Metric, F.Cu at (235.5, 88.9)
- added D8: D, Diode_SMD:D_0805_2012Metric, F.Cu at (209.8, 111.5)
- added J1: Conn_01x01_Female, Connector_PinSocket_2.54mm:PinSocket_1x01_P2.54mm_Vertical, F.Cu at (189.3, 125.7)
- added J10: Conn_01x01_Female, Connector_PinSocket_2.54mm:PinSocket_1x01_P2.54mm_Vertical, F.Cu at (196.0, 121.1)
- added J11: Conn_01x01_Female, Connector_PinSocket_2.54mm:PinSocket_1x01_P2.54mm_Vertical, F.Cu at (209.8, 107.7)
- added J12: Conn_01x01_Female, Connector_PinSocket_2.54mm:PinSocket_1x01_P2.54mm_Vertical, F.Cu at (182.2, 121.1)
- added J13: Conn_01x01_Female, Connector_PinSocket_2.54mm:PinSocket_1x01_P2.54mm_Vertical, F.Cu at (186.8, 121.1)
- added J14: Conn_01x01_Female, Connector_PinSocket_2.54mm:PinSocket_1x01_P2.54mm_Vertical, F.Cu at (180.1, 125.7)
- added J15: Conn_01x01_Female, Connector_PinSocket_2.54mm:PinSocket_1x01_P2.54mm_Vertical, F.Cu at (170.9, 124.4)
- added J16: Conn_01x01_Female, Connector_PinSocket_2.54mm:PinSocket_1x01_P2.54mm_Vertical, F.Cu at (214.4, 103.1)
- added J2: Conn_01x01_Female, Connector_PinSocket_2.54mm:PinSocket_1x01_P2.54mm_Vertical, F.Cu at (191.4, 121.1)
- added J3: Conn_01x01_Female, Connector_PinSocket_2.54mm:PinSocket_1x01_P2.54mm_Vertical, F.Cu at (205.2, 103.1)
- added J4: Conn_01x01_Female, Connector_PinSocket_2.54mm:PinSocket_1x01_P2.54mm_Vertical, F.Cu at (175.5, 124.4)
- added J5: Conn_01x01_Female, Connector_PinSocket_2.54mm:PinSocket_1x01_P2.54mm_Vertical, F.Cu at (205.2, 107.7)
- added J6: Conn_01x01_Female, Connector_PinSocket_2.54mm:PinSocket_1x01_P2.54mm_Vertical, F.Cu at (205.2, 112.3)
- added J7: Conn_01x01_Female, Connector_PinSocket_2.54mm:PinSocket_1x01_P2.54mm_Vertical, F.Cu at (235.6, 85.1)
- added J8: Conn_01x01_Female, Connector_PinSocket_2.54mm:PinSocket_1x01_P2.54mm_Vertical, F.Cu at (209.8, 103.1)
- added J9: Conn_01x01_Female, Connector_PinSocket_2.54mm:PinSocket_1x01_P2.54mm_Vertical, F.Cu at (184.7, 125.7)
- added Q1: Q_NMOS_GDS, Package_TO_SOT_SMD:TO-3P-SideMount, F.Cu at (180.2, 109.8)
- added Q2: Q_NMOS_GDS, Package_TO_SOT_SMD:TO-3P-SideMount, F.Cu at (138.1, 93.0)
- added Q3: Q_NMOS_GDS, Package_TO_SOT_SMD:TO-3P-SideMount, F.Cu at (165.0, 109.8)
- added Q4: Q_NMOS_GDS, Package_TO_SOT_SMD:TO-3P-SideMount, F.Cu at (225.7, 91.8)
- added Q5: Q_NMOS_GDS, Package_TO_SOT_SMD:TO-3P-SideMount, F.Cu at (210.5, 91.8)
- added Q6: Q_NMOS_GDS, Package_TO_SOT_SMD:TO-3P-SideMount, F.Cu at (195.3, 91.8)
- added Q7: Q_NMOS_GDS, Package_TO_SOT_SMD:TO-3P-SideMount, F.Cu at (180.2, 91.8)
- added Q8: Q_NMOS_GDS, Package_TO_SOT_SMD:TO-3P-SideMount, F.Cu at (195.3, 109.8)
- added R1: 5.1, Resistor_SMD:R_1206_3216Metric, F.Cu at (160.2, 120.5)
- added R2: 5.1, Resistor_SMD:R_1206_3216Metric, F.Cu at (165.8, 120.5)
- added R3: 5.1, Resistor_SMD:R_1206_3216Metric, F.Cu at (171.4, 120.5)
- added R4: 5.1, Resistor_SMD:R_1206_3216Metric, F.Cu at (177.0, 120.5)
- added R5: 5.1, Resistor_SMD:R_1206_3216Metric, F.Cu at (165.8, 123.7)
- added R518: 100k, Resistor_SMD:R_0805_2012Metric, F.Cu at (299.5, 57.1)
- added R519: 470, Resistor_SMD:R_0805_2012Metric, F.Cu at (304.1, 52.4)
- added R6: 5.1, Resistor_SMD:R_1206_3216Metric, F.Cu at (160.2, 123.7)
- added R7: 5.1, Resistor_SMD:R_1206_3216Metric, F.Cu at (160.2, 127.0)
- added R8: 5.1, Resistor_SMD:R_1206_3216Metric, F.Cu at (165.8, 127.0)
- added R9: 5.1k, Resistor_SMD:R_0805_2012Metric, F.Cu at (205.1, 116.1)
- added U601: L7809, Package_TO_SOT_SMD:TO-252-2, F.Cu at (251.0, 120.6)
- added U602: L7805, Package_TO_SOT_SMD:TO-252-2, F.Cu at (251.0, 128.7)
- D501, D502, D503, D504, D507, D508: value D -> MBR0530
- D505, D506: value D -> LL4148
- J504: value Conn_01x03_Male -> Conn_01x01_Female; footprint Connector_PinHeader_2.54mm:PinHeader_1x03_P2.54mm_Vertical -> Connector_PinHeader_2.54mm:PinHeader_1x01_P2.54mm_Vertical
- J505: value Conn_01x02_Male -> Screw_Terminal_01x02; footprint Connector_PinHeader_2.54mm:PinHeader_1x02_P2.54mm_Vertical -> TerminalBlock:TerminalBlock_Altech_AK300-2_P5.00mm
- J506: value Conn_01x02_Male -> Conn_01x01_Female; footprint Connector_PinHeader_2.54mm:PinHeader_1x02_P2.54mm_Vertical -> Connector_PinHeader_2.54mm:PinHeader_1x01_P2.54mm_Vertical
- J507: value Conn_01x02_Male -> Conn_01x03_Male; footprint Connector_PinHeader_2.54mm:PinHeader_1x02_P2.54mm_Vertical -> Connector_PinHeader_2.54mm:PinHeader_1x03_P2.54mm_Vertical
- J508, J510: value Conn_01x01_Female -> Conn_01x02_Male; footprint Connector_PinHeader_2.54mm:PinHeader_1x01_P2.54mm_Vertical -> Connector_PinHeader_2.54mm:PinHeader_1x02_P2.54mm_Vertical
- J509: value Screw_Terminal_01x02 -> Conn_01x02_Male; footprint TerminalBlock:TerminalBlock_Altech_AK300-2_P5.00mm -> Connector_PinHeader_2.54mm:PinHeader_1x02_P2.54mm_Vertical
- moved D402 336.4 mm to (295.0, 84.3)
- moved D401 334.1 mm to (290.3, 89.0)
- moved C403 321.9 mm to (278.1, 100.7)
- moved J403 310.0 mm to (290.4, 85.1)
- moved C406 305.8 mm to (279.5, 95.0)
- moved R401 299.5 mm to (271.5, 111.0)
- moved TP501 298.0 mm to (321.6, 25.7)
- moved R505 296.5 mm to (262.8, 28.6)
- moved C503 294.1 mm to (316.2, 34.6)
- moved U505 293.4 mm to (277.3, 39.0)
- moved C401 292.2 mm to (246.8, 98.6)
- moved C402 292.2 mm to (246.8, 88.1)
- moved U506 291.0 mm to (285.7, 42.4)
- moved U504 286.7 mm to (273.5, 57.2)
- moved J401 285.2 mm to (271.6, 107.2)
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Connections:
- net Inverter_source_2 renamed Vbus-
- J501 pad 1: Net-(C509-Pad1) -> Net-(D501-Pad2)
- J502 pad 1: Net-(C509-Pad2) -> Net-(D503-Pad2)
- J502 pad 2: Net-(C509-Pad1) -> Net-(D501-Pad2)
- J503 pad 1: Net-(C509-Pad2) -> Net-(D503-Pad2)
- J504 pad 1: Net-(J504-Pad1) -> Net-(C509-Pad1)
- J505 pad 1: GDT_INB -> Net-(C509-Pad2)
- J505 pad 2: GDT_INA -> Net-(C509-Pad1)
- J506 pad 1: GDT_INA -> Net-(C509-Pad2)
- J507 pad 2: Net-(J507-Pad2) -> Net-(C509-Pad1)
- J508 pad 1: Net-(D501-Pad2) -> GDT_INB
- J509 pad 1: Net-(D503-Pad2) -> GDT_INA
- J509 pad 2: Net-(D501-Pad2) -> GDT_INB
- J510 pad 1: Net-(D503-Pad2) -> Net-(J510-Pad1)
- L501 pad 1: Net-(J504-Pad1) -> Net-(J507-Pad1)
- L501 pad 2: Net-(J504-Pad3) -> Net-(J507-Pad3)
- R505 pad 1: Net-(J504-Pad3) -> Net-(J507-Pad3)
- R517 pad 1: Net-(D509-Pad1) -> Net-(R513-Pad2)
- R517 pad 2: Net-(C515-Pad1) -> Net-(C514-Pad1)
- U505 pad 10: Net-(D509-Pad1) -> Net-(D511-Pad1)
- U506 pad 3: Net-(J507-Pad2) -> Net-(J510-Pad2)
- U506 pad 6: Net-(J507-Pad1) -> Net-(J510-Pad1)
- U506 pad 8: Net-(D509-Pad1) -> Net-(D511-Pad1)
