File: power_regulation.kicad_sch (KiCad schematic)
At the start: 0 parts

Commit message: Update
Parts:
- added C601, C603, C605, C606: 100n, symbol Device:C
- added C602, C604, C607: 470u, symbol Device:C_Polarized_US
- added D601, D602, D603: LED, symbol Device:LED
- added R601, R602, R603: 470, symbol Device:R
- added U601: L7809, symbol Regulator_Linear:L7809
- added U602: L7805, symbol Regulator_Linear:L7805
Connections:
- new net: C601.2, C602.2, C603.2, C604.2, C605.2, C606.2, C607.2, D601.1 (K), D602.1 (K), D603.1 (K), U601.2 (GND), U602.2 (GND)
- new net: D602.2 (A), R602.2
- new net: D603.2 (A), R603.2
- new net: D601.2 (A), R601.2
- new net +5V: C606.1, C607.1, R603.1, U602.3 (OUT)
- new net +9V: C603.1, C604.1, C605.1, R602.1, U601.3 (OUT), U602.1 (IN)
- new net VCC: C601.1, C602.1, R601.1, U601.1 (IN)

Commit message: 0.1V control-circuit
Next relese:
Mounting holes;
Fan header;
Better layout;
Bigger  capacitors;
Parts:
- U601, U602: footprint (none) -> Package_TO_SOT_SMD:TO-252-2
Changed lines of the file:
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@@
     (property "Reference" "U601" (id 0) (at 72.39 33.02 0))
     (property "Value" "L7809" (id 1) (at 72.39 35.56 0))
-    (property "Footprint" "" (id 2) (at 73.025 44.45 0)
+    (property "Footprint" "Package_TO_SOT_SMD:TO-252-2" (id 2) (at 73.025 44.45 0)
       (effects (font (size 1.27 1.27) italic) (justify left) hide)
     )
@@
     (property "Reference" "U602" (id 0) (at 128.905 33.02 0))
     (property "Value" "L7805" (id 1) (at 128.905 35.56 0))
-    (property "Footprint" "" (id 2) (at 129.54 44.45 0)
+    (property "Footprint" "Package_TO_SOT_SMD:TO-252-2" (id 2) (at 129.54 44.45 0)
       (effects (font (size 1.27 1.27) italic) (justify left) hide)
     )
