File: Controller/DRSSTC controller/_autosave-GDT_primary.kicad_sch (KiCad schematic)
At the start: 20 parts, among them J401 Conn_01x01_Female, J402 Screw_Terminal_01x02, J403 Conn_01x01_Female, Q401 Q_PMOS_GDS, Q402 Q_NMOS_GDS, Q403 Q_PMOS_GDS, Q404 Q_NMOS_GDS, U401 UCC27524

Commit message: 0.1V control-circuit
Next relese:
Mounting holes;
Fan header;
Better layout;
Bigger  capacitors;
Parts:
- removed C403: 100n, Capacitor_SMD:C_0805_2012Metric, symbol Device:C
- removed C404: 1u, Capacitor_SMD:C_01005_0402Metric, symbol Device:C
- removed D401, D402: D, Diode_SMD:D_0805_2012Metric, symbol Device:D
- added C1: 4.7u, Capacitor_SMD:C_1206_3216Metric, symbol Device:C
- added C2: 1u, Capacitor_SMD:C_0805_2012Metric, symbol Device:C
- added D1, D2: LL4148, Diode_SMD:D_MiniMELF, symbol Diode:LL4148
- C401, C402: footprint Capacitor_THT:C_Rect_L16.5mm_W9.0mm_P15.00mm_MKT -> Capacitor_SMD:C_1206_3216Metric
- C405, C407: footprint Capacitor_SMD:C_01005_0402Metric -> Capacitor_SMD:C_0805_2012Metric
- C406: footprint Capacitor_SMD:C_1825_4564Metric -> Capacitor_SMD:C_2220_5650Metric
- J402: footprint TerminalBlock:TerminalBlock_Altech_AK300-2_P5.00mm -> TerminalBlock_Phoenix:TerminalBlock_Phoenix_PT-1,5-2-3.5-H_1x02_P3.50mm_Horizontal
- U401: footprint TestPoint:TestPoint_Loop_D2.50mm_Drill1.0mm -> Package_SO:SOIC-8_3.9x4.9mm_P1.27mm
Connections:
- net +9V: now also C1.1
- net GND: now also C1.2
- net VCC: now also D1.1 (K), D2.1 (K)
- net TopSide_PGate: now reaches Q401.1 (G), R401.2
- net TopSide_PGate: now also C2.1, D1.2 (A)
- net BottomSide_PGate: now reaches C405.1, Q403.1 (G), R402.2
- net BottomSide_PGate: now also D2.2 (A)
- net GDT_terminal_A: now reaches J402.2 (Pin_2), J403.1 (Pin_1), Q403.2 (D), Q404.2 (D)
- net BottomSide_NGate: now reaches C405.2, Q404.1 (G), U401.8 (OUTB)
- net TopSide_NGate: now reaches Q402.1 (G), U401.6 (OUTA)
- net TopSide_NGate: now also C2.2
- net GDT_terminal_B: now reaches C406.2, C407.2, J401.1 (Pin_1), J402.1 (Pin_1)
Changed lines of the file:
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@@
     )
   )
-  (symbol (lib_id "Device:C") (at 86.995 149.86 0) (unit 1)
-    (in_bom yes) (on_board yes)
-    (property "Reference" "C403" (id 0) (at 87.63 147.32 0)
-      (effects (font (size 1.27 1.27)) (justify left))
-    )
-    (property "Value" "100n" (id 1) (at 87.63 152.4 0)
-      (effects (font (size 1.27 1.27)) (justify left))
-    )
-    (property "Footprint" "Capacitor_SMD:C_0805_2012Metric" (id 2) (at 87.9602 153.67 0)
-      (effects (font (size 1.27 1.27)) hide)
-    )
-    (property "Datasheet" "~" (id 3) (at 86.995 149.86 0)
-      (effects (font (size 1.27 1.27)) hide)
-    )
-    (pin "1")
-    (pin "2")
+  (hierarchical_label "GDT_terminal_A" (shape input) (at 180.34 102.235 0)
+    (effects (font (size 1.27 1.27)) (justify left))
+  )
+  (hierarchical_label "TopSide_NGate" (shape input) (at 93.98 66.04 180)
+    (effects (font (size 1.27 1.27)) (justify right))
+  )
+  (hierarchical_label "BottomSide_NGate" (shape input) (at 93.98 109.22 180)
+    (effects (font (size 1.27 1.27)) (justify right))
+  )
+  (hierarchical_label "TopSide_PGate" (shape input) (at 106.68 52.705 180)
+    (effects (font (size 1.27 1.27)) (justify right))
+  )
+  (hierarchical_label "BottomSide_PGate" (shape input) (at 106.68 95.885 180)
+    (effects (font (size 1.27 1.27)) (justify right))
+  )
+  (hierarchical_label "GDT_terminal_B" (shape input) (at 180.34 59.055 0)
+    (effects (font (size 1.27 1.27)) (justify left))
   )
   (symbol (lib_id "Device:Q_PMOS_GDS") (at 130.175 52.705 0) (mirror x) (unit 1)
@@
     (pin "3")
   )
-  (symbol (lib_id "Device:D") (at 106.68 46.99 270) (unit 1)
-    (in_bom yes) (on_board yes) (fields_autoplaced)
-    (property "Reference" "D401" (id 0) (at 109.22 45.7199 90)
-      (effects (font (size 1.27 1.27)) (justify left))
-    )
-    (property "Value" "D" (id 1) (at 109.22 48.2599 90)
-      (effects (font (size 1.27 1.27)) (justify left))
-    )
-    (property "Footprint" "Diode_SMD:D_0805_2012Metric" (id 2) (at 106.68 46.99 0)
-      (effects (font (size 1.27 1.27)) hide)
-    )
-    (property "Datasheet" "~" (id 3) (at 106.68 46.99 0)
-      (effects (font (size 1.27 1.27)) hide)
-    )
-    (pin "1")
-    (pin "2")
-  )
   (symbol (lib_id "Device:C") (at 71.755 149.86 0) (unit 1)
     (in_bom yes) (on_board yes)
@@
       (effects (font (size 1.27 1.27)) (justify left))
     )
-    (property "Footprint" "Capacitor_THT:C_Rect_L16.5mm_W9.0mm_P15.00mm_MKT" (id 2) (at 72.7202 153.67 0)
+    (property "Footprint" "Capacitor_SMD:C_1206_3216Metric" (id 2) (at 72.7202 153.67 0)
       (effects (font (size 1.27 1.27)) hide)
     )
@@
     (pin "2")
   )
+  (symbol (lib_id "Diode:LL4148") (at 106.68 90.17 270) (unit 1)
+    (in_bom yes) (on_board yes) (fields_autoplaced)
+    (property "Reference" "D2" (id 0) (at 109.22 88.8999 90)
+      (effects (font (size 1.27 1.27)) (justify left))
+    )
+    (property "Value" "LL4148" (id 1) (at 109.22 91.4399 90)
+      (effects (font (size 1.27 1.27)) (justify left))
+    )
+    (property "Footprint" "Diode_SMD:D_MiniMELF" (id 2) (at 102.235 90.17 0)
+      (effects (font (size 1.27 1.27)) hide)
+    )
+    (property "Datasheet" "http://www.vishay.com/docs/85557/ll4148.pdf" (id 3) (at 106.68 90.17 0)
+      (effects (font (size 1.27 1.27)) hide)
+    )
+    (pin "1")
+    (pin "2")
+  )
   (symbol (lib_id "Device:C") (at 106.68 101.6 0) (unit 1)
     (in_bom yes) (on_board yes) (fields_autoplaced)
@@
       (effects (font (size 1.27 1.27)) (justify left))
     )
-    (property "Footprint" "Capacitor_SMD:C_01005_0402Metric" (id 2) (at 107.6452 105.41 0)
+    (property "Footprint" "Capacitor_SMD:C_0805_2012Metric" (id 2) (at 107.6452 105.41 0)
       (effects (font (size 1.27 1.27)) hide)
     )
@@
     (pin "2")
     (pin "3")
-  )
-  (symbol (lib_id "Device:C") (at 106.68 58.42 0) (unit 1)
-    (in_bom yes) (on_board yes) (fields_autoplaced)
-    (property "Reference" "C404" (id 0) (at 110.49 57.1499 0)
-      (effects (font (size 1.27 1.27)) (justify left))
-    )
-    (property "Value" "1u" (id 1) (at 110.49 59.6899 0)
-      (effects (font (size 1.27 1.27)) (justify left))
-    )
-    (property "Footprint" "Capacitor_SMD:C_01005_0402Metric" (id 2) (at 107.6452 62.23 0)
-      (effects (font (size 1.27 1.27)) hide)
-    )
-    (property "Datasheet" "~" (id 3) (at 106.68 58.42 0)
-      (effects (font (size 1.27 1.27)) hide)
-    )
-    (pin "1")
-    (pin "2")
   )
   (symbol (lib_id "Device:C") (at 161.29 59.055 90) (unit 1)
@@
     (property "Reference" "C406" (id 0) (at 161.29 55.88 90))
     (property "Value" "2.2u" (id 1) (at 161.29 62.23 90))
-    (property "Footprint" "Capacitor_SMD:C_1825_4564Metric" (id 2) (at 165.1 58.0898 0)
+    (property "Footprint" "Capacitor_SMD:C_2220_5650Metric" (id 2) (at 165.1 58.0898 0)
       (effects (font (size 1.27 1.27)) hide)
     )
@@
       (effects (font (size 1.27 1.27)) (justify left))
     )
-    (property "Footprint" "TerminalBlock:TerminalBlock_Altech_AK300-2_P5.00mm" (id 2) (at 191.135 76.835 0)
+    (property "Footprint" "TerminalBlock_Phoenix:TerminalBlock_Phoenix_PT-1,5-2-3.5-H_1x02_P3.50mm_Horizontal" (id 2) (at 191.135 76.835 0)
       (effects (font (size 1.27 1.27)) hide)
     )
@@
       (effects (font (size 1.27 1.27)) (justify left))
     )
-    (property "Footprint" "Capacitor_THT:C_Rect_L16.5mm_W9.0mm_P15.00mm_MKT" (id 2) (at 63.8302 153.67 0)
+    (property "Footprint" "Capacitor_SMD:C_1206_3216Metric" (id 2) (at 63.8302 153.67 0)
       (effects (font (size 1.27 1.27)) hide)
     )
@@
     (property "Reference" "U401" (id 0) (at 72.39 76.835 0))
     (property "Value" "UCC27524" (id 1) (at 72.39 92.075 0))
-    (property "Footprint" "TestPoint:TestPoint_Loop_D2.50mm_Drill1.0mm" (id 2) (at 69.85 85.725 0)
-      (effects (font (size 1.27 1.27)) hide)
-    )
-    (property "Datasheet" "" (id 3) (at 69.85 85.725 0)
+    (property "Footprint" "Package_SO:SOIC-8_3.9x4.9mm_P1.27mm" (id 2) (at 72.39 93.98 0)
+      (effects (font (size 1.27 1.27)) hide)
+    )
+    (property "Datasheet" "https://datasheet.lcsc.com/lcsc/1912111437_Texas-Instruments-UCC27524DR_C465729.pdf" (id 3) (at 69.85 85.725 0)
       (effects (font (size 1.27 1.27)) hide)
     )
@@
     (pin "8")
   )
-  (symbol (lib_id "Device:D") (at 106.68 90.17 270) (unit 1)
-    (in_bom yes) (on_board yes) (fields_autoplaced)
-    (property "Reference" "D402" (id 0) (at 109.22 88.8999 90)
-      (effects (font (size 1.27 1.27)) (justify left))
-    )
-    (property "Value" "D" (id 1) (at 109.22 91.4399 90)
-      (effects (font (size 1.27 1.27)) (justify left))
-    )
-    (property "Footprint" "Diode_SMD:D_0805_2012Metric" (id 2) (at 106.68 90.17 0)
-      (effects (font (size 1.27 1.27)) hide)
-    )
-    (property "Datasheet" "~" (id 3) (at 106.68 90.17 0)
+  (symbol (lib_id "Device:C") (at 106.68 58.42 0) (unit 1)
+    (in_bom yes) (on_board yes) (fields_autoplaced)
+    (property "Reference" "C2" (id 0) (at 110.49 57.1499 0)
+      (effects (font (size 1.27 1.27)) (justify left))
+    )
+    (property "Value" "1u" (id 1) (at 110.49 59.6899 0)
+      (effects (font (size 1.27 1.27)) (justify left))
+    )
+    (property "Footprint" "Capacitor_SMD:C_0805_2012Metric" (id 2) (at 107.6452 62.23 0)
+      (effects (font (size 1.27 1.27)) hide)
+    )
+    (property "Datasheet" "~" (id 3) (at 106.68 58.42 0)
+      (effects (font (size 1.27 1.27)) hide)
+    )
+    (pin "1")
+    (pin "2")
+  )
+  (symbol (lib_id "Diode:LL4148") (at 106.68 46.99 270) (unit 1)
+    (in_bom yes) (on_board yes) (fields_autoplaced)
+    (property "Reference" "D1" (id 0) (at 109.22 45.7199 90)
+      (effects (font (size 1.27 1.27)) (justify left))
+    )
+    (property "Value" "LL4148" (id 1) (at 109.22 48.2599 90)
+      (effects (font (size 1.27 1.27)) (justify left))
+    )
+    (property "Footprint" "Diode_SMD:D_MiniMELF" (id 2) (at 102.235 46.99 0)
+      (effects (font (size 1.27 1.27)) hide)
+    )
+    (property "Datasheet" "http://www.vishay.com/docs/85557/ll4148.pdf" (id 3) (at 106.68 46.99 0)
       (effects (font (size 1.27 1.27)) hide)
     )
@@
     (pin "1")
   )
+  (symbol (lib_id "Device:C") (at 86.995 149.86 0) (unit 1)
+    (in_bom yes) (on_board yes)
+    (property "Reference" "C1" (id 0) (at 87.63 147.32 0)
+      (effects (font (size 1.27 1.27)) (justify left))
+    )
+    (property "Value" "4.7u" (id 1) (at 87.63 152.4 0)
+      (effects (font (size 1.27 1.27)) (justify left))
+    )
+    (property "Footprint" "Capacitor_SMD:C_1206_3216Metric" (id 2) (at 87.9602 153.67 0)
+      (effects (font (size 1.27 1.27)) hide)
+    )
+    (property "Datasheet" "~" (id 3) (at 86.995 149.86 0)
+      (effects (font (size 1.27 1.27)) hide)
+    )
+    (pin "1")
+    (pin "2")
+  )
   (symbol (lib_id "Device:C") (at 165.1 53.975 90) (unit 1)
     (in_bom yes) (on_board yes) (fields_autoplaced)
     (property "Reference" "C407" (id 0) (at 165.1 46.99 90))
     (property "Value" "1u" (id 1) (at 165.1 49.53 90))
-    (property "Footprint" "Capacitor_SMD:C_01005_0402Metric" (id 2) (at 168.91 53.0098 0)
-      (effects (font (size 1.27 1.27)) hide)
-    )
+    (property "Footprint" "Capacitor_SMD:C_0805_2012Metric" (id 2) (at 168.91 53.0098 0)
+      (effects (font (size 1.27 1.27)) hide)
+    )

Commit message: V0.15a
Parts:
- Q401, Q402, Q403, Q404: footprint Package_TO_SOT_SMD:TO-252-3_TabPin2 -> Package_TO_SOT_SMD:TO-252-2
Changed lines of the file:
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@@
       (effects (font (size 1.27 1.27)) (justify left))
     )
-    (property "Footprint" "Package_TO_SOT_SMD:TO-252-3_TabPin2" (id 2) (at 135.255 55.245 0)
+    (property "Footprint" "Package_TO_SOT_SMD:TO-252-2" (id 2) (at 135.255 55.245 0)
       (effects (font (size 1.27 1.27)) hide)
     )
@@
       (effects (font (size 1.27 1.27)) (justify left))
     )
-    (property "Footprint" "Package_TO_SOT_SMD:TO-252-3_TabPin2" (id 2) (at 135.255 98.425 0)
+    (property "Footprint" "Package_TO_SOT_SMD:TO-252-2" (id 2) (at 135.255 98.425 0)
       (effects (font (size 1.27 1.27)) hide)
     )
@@
       (effects (font (size 1.27 1.27)) (justify left))
     )
-    (property "Footprint" "Package_TO_SOT_SMD:TO-252-3_TabPin2" (id 2) (at 135.255 63.5 0)
+    (property "Footprint" "Package_TO_SOT_SMD:TO-252-2" (id 2) (at 135.255 63.5 0)
       (effects (font (size 1.27 1.27)) hide)
     )
@@
       (effects (font (size 1.27 1.27)) (justify left))
     )
-    (property "Footprint" "Package_TO_SOT_SMD:TO-252-3_TabPin2" (id 2) (at 135.255 106.68 0)
-      (effects (font (size 1.27 1.27)) hide)
-    )
+    (property "Footprint" "Package_TO_SOT_SMD:TO-252-2" (id 2) (at 135.255 106.68 0)
+      (effects (font (size 1.27 1.27)) hide)
+    )
