File: Controller/DRSSTC controller/_autosave-Physical.kicad_sch (KiCad schematic)
At the start: 4 parts

Commit message: V0.15a
Parts:
- H1, H2, H3, H4: renamed from H?; footprint (none) -> MountingHole:MountingHole_3.2mm_M3
Changed lines of the file:
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@@
   (symbol (lib_id "Mechanical:MountingHole") (at 48.26 60.96 0) (unit 1)
     (in_bom yes) (on_board yes) (fields_autoplaced)
-    (property "Reference" "H?" (id 0) (at 51.435 59.6899 0)
+    (property "Reference" "H1" (id 0) (at 51.435 59.6899 0)
       (effects (font (size 1.27 1.27)) (justify left))
     )
@@
       (effects (font (size 1.27 1.27)) (justify left))
     )
-    (property "Footprint" "" (id 2) (at 48.26 60.96 0)
+    (property "Footprint" "MountingHole:MountingHole_3.2mm_M3" (id 2) (at 48.26 60.96 0)
       (effects (font (size 1.27 1.27)) hide)
     )
@@
   (symbol (lib_id "Mechanical:MountingHole") (at 113.665 60.96 0) (unit 1)
     (in_bom yes) (on_board yes) (fields_autoplaced)
-    (property "Reference" "H?" (id 0) (at 116.84 59.6899 0)
+    (property "Reference" "H4" (id 0) (at 116.84 59.6899 0)
       (effects (font (size 1.27 1.27)) (justify left))
     )
@@
       (effects (font (size 1.27 1.27)) (justify left))
     )
-    (property "Footprint" "" (id 2) (at 113.665 60.96 0)
+    (property "Footprint" "MountingHole:MountingHole_3.2mm_M3" (id 2) (at 113.665 60.96 0)
       (effects (font (size 1.27 1.27)) hide)
     )
@@
   (symbol (lib_id "Mechanical:MountingHole") (at 93.345 60.96 0) (unit 1)
     (in_bom yes) (on_board yes) (fields_autoplaced)
-    (property "Reference" "H?" (id 0) (at 96.52 59.6899 0)
+    (property "Reference" "H3" (id 0) (at 96.52 59.6899 0)
       (effects (font (size 1.27 1.27)) (justify left))
     )
@@
       (effects (font (size 1.27 1.27)) (justify left))
     )
-    (property "Footprint" "" (id 2) (at 93.345 60.96 0)
+    (property "Footprint" "MountingHole:MountingHole_3.2mm_M3" (id 2) (at 93.345 60.96 0)
       (effects (font (size 1.27 1.27)) hide)
     )
@@
   (symbol (lib_id "Mechanical:MountingHole") (at 69.85 60.96 0) (unit 1)
     (in_bom yes) (on_board yes) (fields_autoplaced)
-    (property "Reference" "H?" (id 0) (at 73.025 59.6899 0)
+    (property "Reference" "H2" (id 0) (at 73.025 59.6899 0)
       (effects (font (size 1.27 1.27)) (justify left))
     )
@@
       (effects (font (size 1.27 1.27)) (justify left))
     )
-    (property "Footprint" "" (id 2) (at 69.85 60.96 0)
+    (property "Footprint" "MountingHole:MountingHole_3.2mm_M3" (id 2) (at 69.85 60.96 0)
       (effects (font (size 1.27 1.27)) hide)
     )
