File: Controller/DRSSTC controller/_autosave-Power_regulation.kicad_sch (KiCad schematic)
At the start: 23 parts, among them J7 Conn_01x01_Female, J8 Screw_Terminal_01x02, J9 Conn_01x01_Female, U601 L7809, U602 L7805

Commit message: V0.15a
Parts:
- J10: renamed from J?; footprint (none) -> Connector_PinHeader_2.54mm:PinHeader_1x02_P2.54mm_Vertical
- U1: renamed from U?; footprint (none) -> Package_TO_SOT_SMD:TO-252-2
- gave numbers to parts that had none: 3
Changed lines of the file:
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@@
   (symbol (lib_id "power:VCC") (at 53.34 130.175 0) (unit 1)
     (in_bom yes) (on_board yes) (fields_autoplaced)
-    (property "Reference" "#PWR?" (id 0) (at 53.34 133.985 0)
+    (property "Reference" "#PWR0104" (id 0) (at 53.34 133.985 0)
       (effects (font (size 1.27 1.27)) hide)
     )
@@
   (symbol (lib_id "Device:C") (at 76.835 141.605 0) (unit 1)
     (in_bom yes) (on_board yes)
-    (property "Reference" "C?" (id 0) (at 77.47 139.065 0)
+    (property "Reference" "C4" (id 0) (at 77.47 139.065 0)
       (effects (font (size 1.27 1.27)) (justify left))
     )
@@
   (symbol (lib_id "Connector:Conn_01x02_Male") (at 99.695 142.24 180) (unit 1)
     (in_bom yes) (on_board yes) (fields_autoplaced)
-    (property "Reference" "J?" (id 0) (at 100.965 139.6999 0)
+    (property "Reference" "J10" (id 0) (at 100.965 139.6999 0)
       (effects (font (size 1.27 1.27)) (justify right))
     )
@@
       (effects (font (size 1.27 1.27)) (justify right))
     )
-    (property "Footprint" "" (id 2) (at 99.695 142.24 0)
+    (property "Footprint" "Connector_PinHeader_2.54mm:PinHeader_1x02_P2.54mm_Vertical" (id 2) (at 99.695 142.24 0)
       (effects (font (size 1.27 1.27)) hide)
     )
@@
   (symbol (lib_id "power:+12V") (at 81.28 130.175 0) (unit 1)
     (in_bom yes) (on_board yes) (fields_autoplaced)
-    (property "Reference" "#PWR?" (id 0) (at 81.28 133.985 0)
+    (property "Reference" "#PWR0103" (id 0) (at 81.28 133.985 0)
       (effects (font (size 1.27 1.27)) hide)
     )
@@
   (symbol (lib_id "Device:C_Polarized_US") (at 85.725 141.605 0) (unit 1)
     (in_bom yes) (on_board yes)
-    (property "Reference" "C?" (id 0) (at 86.36 139.065 0)
+    (property "Reference" "C5" (id 0) (at 86.36 139.065 0)
       (effects (font (size 1.27 1.27)) (justify left))
     )
@@
   (symbol (lib_id "power:GND") (at 67.31 150.495 0) (unit 1)
     (in_bom yes) (on_board yes) (fields_autoplaced)
-    (property "Reference" "#PWR?" (id 0) (at 67.31 156.845 0)
+    (property "Reference" "#PWR0102" (id 0) (at 67.31 156.845 0)
       (effects (font (size 1.27 1.27)) hide)
     )
@@
   (symbol (lib_id "Device:C") (at 53.34 141.605 0) (unit 1)
     (in_bom yes) (on_board yes)
-    (property "Reference" "C?" (id 0) (at 53.975 139.065 0)
+    (property "Reference" "C3" (id 0) (at 53.975 139.065 0)
       (effects (font (size 1.27 1.27)) (justify left))
     )
@@
   (symbol (lib_id "Regulator_Linear:L7812") (at 67.31 133.985 0) (unit 1)
     (in_bom yes) (on_board yes) (fields_autoplaced)
-    (property "Reference" "U?" (id 0) (at 67.31 127 0))
+    (property "Reference" "U1" (id 0) (at 67.31 127 0))
     (property "Value" "L7812" (id 1) (at 67.31 129.54 0))
-    (property "Footprint" "" (id 2) (at 67.945 137.795 0)
+    (property "Footprint" "Package_TO_SOT_SMD:TO-252-2" (id 2) (at 67.945 137.795 0)
       (effects (font (size 1.27 1.27) italic) (justify left) hide)
     )
