File: Controller/DRSSTC controller/DRSSTC controller.kicad_sch (KiCad schematic)
At the start: 0 parts

Commit message: V0.2a
Other:
- company: (none) -> Politehnika
- title: (none) -> DRSSTC controller
Changed lines of the file:
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@@
 (kicad_sch (version 20211123) (generator eeschema)
   (paper "A4")
+  (title_block
+    (title "DRSSTC controller")
+    (date "2023-03-07")
+    (rev "0.2")
+    (company "Politehnika")
+  )
   (sheet (at 31.75 91.44) (size 50.8 26.67) (fields_autoplaced)
     (stroke (width 0.1524) (type solid) (color 0 0 0 0))
