File: Full Bridge/Full Bridge/Full Bridge.kicad_sch (KiCad schematic)
At the start: 49 parts, among them J1 Conn_01x01_Female, J10 Conn_01x01_Female, J11 Conn_01x01_Female, J12 Conn_01x01_Female, J13 Conn_01x01_Female, J14 Conn_01x01_Female, J15 Conn_01x01_Female, J16 Conn_01x01_Female, J2 Conn_01x01_Female, J3 Conn_01x01_Female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

Commit message: v0.2b
Other:
- company: (none) -> Politehnika
- title: (none) -> DRSSTC Full Bridge
Changed lines of the file:
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@@
 (kicad_sch (version 20211123) (generator eeschema)
   (paper "A4")
+  (title_block
+    (title "DRSSTC Full Bridge")
+    (date "2023-03-07")
+    (rev "0.2")
+    (company "Politehnika")
+  )
   (junction (at 71.12 102.87) (diameter 0) (color 0 0 0 0)
   )
